File: garage-dry.kicad_pcb (KiCad board)
At the start: 2 copper layers, 77.5 x 32 mm, 16 parts, among them J1 DOOR OPENER, J2 DC IN, J3 CONTACT, J4 HC-SR04, K1 5V RELAY, Q1 2N3904, U1 XIAO-ESP32-C6-SMD

Commit message: Ready for prod.
Parts:
- K1: value 5V RELAY -> ~
- moved R2 9.60 mm to (167.6, 55.0)
Connections:
- J1 pad 2: GND -> Net-(J1-Pin_2)
- K1 pad 1: (no net) -> Net-(J1-Pin_2)
- K1 pad 2: (no net) -> +5V
- K1 pad 3: (no net) -> unconnected-(K1-Pad3)
- K1 pad 4: (no net) -> Net-(J1-Pin_1)
- K1 pad 5: (no net) -> Net-(D1-A)
- U1 pad 10: DOOR_OPENER -> DOOR_SENSOR
- U1 pad 11: ECHO -> DOOR_OPENER
- U1 pad 8: TRIGGER -> ECHO
- U1 pad 9: DOOR_SENSOR -> TRIGGER
Routing:
- net Net-(J1-Pin_1): track 0.00 -> 32.5 mm, vias 0 -> 1
- net ECHO: track 70.9 -> 41.6 mm, vias 2 -> 0
- net Net-(J1-Pin_2): track 0.00 -> 20.1 mm
- net Net-(D1-A): track 15.4 -> 34.5 mm
- net +5V: track 67.6 -> 84.5 mm
- net DOOR_SENSOR: track 31.6 -> 20.9 mm
- net Net-(J3-Pin_2): track 32.0 -> 41.6 mm
- net TRIGGER: track 42.3 -> 39.6 mm
- net DOOR_OPENER: track 7.80 -> 6.75 mm
- added copper zone on B.Cu, net GND
Other:
- board text added: "SIMPLE GARAGE DOOR OPENER CAMERON-MORGAN.COM V1.2"
- board text removed: "SIMPLE GARAGE DOOR OPENER CAMERON-MORGAN.COM | V1.2"
