File: garage-dry.kicad_sch (KiCad schematic)
At the start: 12 parts, among them J1 DOOR OPENER, J2 DC IN, J3 CONTACT, J4 HC-SR04, K1 5V RELAY, Q1 2N3904, U1 XIAO-ESP32-C6-SMD

Commit message: Ready for prod.
Parts:
- removed K1: 5V RELAY, footprints:RELAY6_S55-5V_CUD, symbol Relay:Relay_SPDT
- added K1: (no value), footprints:RELAY6_S55-5V_CUD, symbol Relay:SR5-5V
Connections:
- net +5V: now also K1.2
- net DOOR_OPENER: now also U1.11 (D10); no longer U1.10 (D9)
- net DOOR_SENSOR: now also U1.10 (D9); no longer U1.9 (D8)
- net ECHO: now also U1.8 (D7); no longer U1.11 (D10)
- net GND: no longer J1.2 (Pin_2)
- net TRIGGER: now also U1.9 (D8); no longer U1.8 (D7)
- net at J1.1 (Pin_1): now also K1.4
- net at D1.2 (A), Q1.3 (C): now also K1.5
- new net: J1.2 (Pin_2), K1.1
Other:
- moved on the sheet: J1
